Commit message: 从本地wheel_legged_genesis_clean目录添加所有assets文件
- 添加完整的assets目录结构
- 包括所有URDF、STL、OBJ、XML文件
- 修复路径引用一致性
- 确保项目可以正确加载所有资源文件

File: assets/description/meshes/wheel_leg.urdf (robot description, URDF)
Before this commit: robot wheel_leg, 7 links, 6 joints
Links:
- link L1_link: geometry collision mesh filename=package://description/meshes/L1_link.STL; visual mesh filename=package://description/meshes/L1_link.STL
- link L2_link: geometry collision mesh filename=package://description/meshes/L2_link.STL; visual mesh filename=package://description/meshes/L2_link.STL
- link L3_link: geometry collision mesh filename=package://description/meshes/L3_link.STL; visual mesh filename=package://description/meshes/L3_link.STL
- link R1_link: geometry collision mesh filename=package://description/meshes/R1_link.STL; visual mesh filename=package://description/meshes/R1_link.STL
- link R2_link: geometry collision mesh filename=package://description/meshes/R2_link.STL; visual mesh filename=package://description/meshes/R2_link.STL
- link R3_link: geometry collision mesh filename=package://description/meshes/R3_link.STL; visual mesh filename=package://description/meshes/R3_link.STL
- link base_link: geometry collision mesh filename=package://description/meshes/base_link.STL; visual mesh filename=package://description/meshes/base_link.STL

File: assets/terrain/plane/plane_light.urdf (robot description, URDF)
Before this commit: robot plane, 1 links, 0 joints
Links:
- link planeLink: mass 1.0 -> .0; geometry collision box size=200 200 10; visual mesh filename=plane100_light.obj scale=1 1 1

File: assets/urdf/wheel_leg/meshes/wheel_leg2.urdf (robot description, URDF)
Before this commit: robot wheel_leg, 7 links, 6 joints
Links:
- added link world
Joints:
- added joint floating_base_joint: type floating, parent world, child base_link
